Commit message: updated GPSR gazebo map

File: src/robot_description/urdf/arm/rx200.urdf.xacro (robot description, xacro)
@@ -15,5 +15,5 @@
   </xacro:if>
   <material name="interbotix_black">
-    <texture filename="package://interbotix_xsarm_descriptions/meshes/interbotix_black.png"/>
+    <texture filename="package://robot_description/meshes/arm/arm/interbotix_black.png"/>
   </material>
   <xacro:if value="$(arg use_world_frame)">
@@ -28,5 +28,5 @@
       <origin rpy="0 0 ${-pi/2}" xyz="0 0 0"/>
       <geometry>
-        <mesh filename="package://interbotix_xsarm_descriptions/meshes/rx200_meshes/rx200_1_base.stl" scale="0.001 0.001 0.001"/>
+        <mesh filename="package://robot_description/meshes/arm/arm/rx200_meshes/rx200_1_base.stl" scale="0.001 0.001 0.001"/>
       </geometry>
       <material name="interbotix_black"/>
@@ -35,5 +35,5 @@
       <origin rpy="0 0 ${-pi/2}" xyz="0 0 0"/>
       <geometry>
-        <mesh filename="package://interbotix_xsarm_descriptions/meshes/rx200_meshes/rx200_1_base.stl" scale="0.001 0.001 0.001"/>
+        <mesh filename="package://robot_description/meshes/arm/arm/rx200_meshes/rx200_1_base.stl" scale="0.001 0.001 0.001"/>
       </geometry>
     </collision>
@@ -65,5 +65,5 @@
       <origin rpy="0 0 ${-pi/2}" xyz="0 0 0.0015"/>
       <geometry>
-        <mesh filename="package://interbotix_xsarm_descriptions/meshes/rx200_meshes/rx200_2_shoulder.stl" scale="0.001 0.001 0.001"/>
+        <mesh filename="package://robot_description/meshes/arm/arm/rx200_meshes/rx200_2_shoulder.stl" scale="0.001 0.001 0.001"/>
       </geometry>
       <material name="interbotix_black"/>
@@ -72,5 +72,5 @@
       <origin rpy="0 0 ${-pi/2}" xyz="0 0 0.0015"/>
       <geometry>
-        <mesh filename="package://interbotix_xsarm_descriptions/meshes/rx200_meshes/rx200_2_shoulder.stl" scale="0.001 0.001 0.001"/>
+        <mesh filename="package://robot_description/meshes/arm/arm/rx200_meshes/rx200_2_shoulder.stl" scale="0.001 0.001 0.001"/>
       </geometry>
     </collision>
@@ -102,12 +102,12 @@
       <origin rpy="0 0 ${pi/2}" xyz="0 0 0"/>
       <geometry>
-        <mesh filename="package://interbotix_xsarm_descriptions/meshes/rx200_meshes/rx200_3_upper_arm.stl" scale="0.001 0.001 0.001"/>
-      </geometry>
-      <material name="interbotix_black"/>
-    </visual>
-    <collision>
-      <origin rpy="0 0 ${pi/2}" xyz="0 0 0"/>
-      <geometry>
-        <mesh filename="package://interbotix_xsarm_descriptions/meshes/rx200_meshes/rx200_3_upper_arm.stl" scale="0.001 0.001 0.001"/>
+        <mesh filename="package://robot_description/meshes/arm/arm/rx200_meshes/rx200_3_upper_arm.stl" scale="0.001 0.001 0.001"/>
+      </geometry>
+      <material name="interbotix_black"/>
+    </visual>
+    <collision>
+      <origin rpy="0 0 ${pi/2}" xyz="0 0 0"/>
+      <geometry>
+        <mesh filename="package://robot_description/meshes/arm/arm/rx200_meshes/rx200_3_upper_arm.stl" scale="0.001 0.001 0.001"/>
       </geometry>
     </collision>
@@ -139,12 +139,12 @@
       <origin rpy="0 0 ${pi/2}" xyz="0 0 0"/>
       <geometry>
-        <mesh filename="package://interbotix_xsarm_descriptions/meshes/rx200_meshes/rx200_4_forearm.stl" scale="0.001 0.001 0.001"/>
-      </geometry>
-      <material name="interbotix_black"/>
-    </visual>
-    <collision>
-      <origin rpy="0 0 ${pi/2}" xyz="0 0 0"/>
-      <geometry>
-        <mesh filename="package://interbotix_xsarm_descriptions/meshes/rx200_meshes/rx200_4_forearm.stl" scale="0.001 0.001 0.001"/>
+        <mesh filename="package://robot_description/meshes/arm/arm/rx200_meshes/rx200_4_forearm.stl" scale="0.001 0.001 0.001"/>
+      </geometry>
+      <material name="interbotix_black"/>
+    </visual>
+    <collision>
+      <origin rpy="0 0 ${pi/2}" xyz="0 0 0"/>
+      <geometry>
+        <mesh filename="package://robot_description/meshes/arm/arm/rx200_meshes/rx200_4_forearm.stl" scale="0.001 0.001 0.001"/>
       </geometry>
     </collision>
@@ -176,12 +176,12 @@
       <origin rpy="0 0 ${pi/2}" xyz="0 0 0"/>
       <geometry>
-        <mesh filename="package://interbotix_xsarm_descriptions/meshes/rx200_meshes/rx200_5_wrist.stl" scale="0.001 0.001 0.001"/>
-      </geometry>
-      <material name="interbotix_black"/>
-    </visual>
-    <collision>
-      <origin rpy="0 0 ${pi/2}" xyz="0 0 0"/>
-      <geometry>
-        <mesh filename="package://interbotix_xsarm_descriptions/meshes/rx200_meshes/rx200_5_wrist.stl" scale="0.001 0.001 0.001"/>
+        <mesh filename="package://robot_description/meshes/arm/arm/rx200_meshes/rx200_5_wrist.stl" scale="0.001 0.001 0.001"/>
+      </geometry>
+      <material name="interbotix_black"/>
+    </visual>
+    <collision>
+      <origin rpy="0 0 ${pi/2}" xyz="0 0 0"/>
+      <geometry>
+        <mesh filename="package://robot_description/meshes/arm/arm/rx200_meshes/rx200_5_wrist.stl" scale="0.001 0.001 0.001"/>
       </geometry>
     </collision>
@@ -213,5 +213,5 @@
       <origin rpy="0 0 ${pi/2}" xyz="-0.02 0 0"/>
       <geometry>
-        <mesh filename="package://interbotix_xsarm_descriptions/meshes/rx200_meshes/rx200_6_gripper.stl" scale="0.001 0.001 0.001"/>
+        <mesh filename="package://robot_description/meshes/arm/arm/rx200_meshes/rx200_6_gripper.stl" scale="0.001 0.001 0.001"/>
       </geometry>
       <material name="interbotix_black"/>
@@ -220,5 +220,5 @@
       <origin rpy="0 0 ${pi/2}" xyz="-0.02 0 0"/>
       <geometry>
-        <mesh filename="package://interbotix_xsarm_descriptions/meshes/rx200_meshes/rx200_6_gripper.stl" scale="0.001 0.001 0.001"/>
+        <mesh filename="package://robot_description/meshes/arm/arm/rx200_meshes/rx200_6_gripper.stl" scale="0.001 0.001 0.001"/>
       </geometry>
     </collision>
@@ -262,5 +262,5 @@
       <origin rpy="0 0 ${pi/2}" xyz="-0.0685 0 0"/>
       <geometry>
-        <mesh filename="package://interbotix_xsarm_descriptions/meshes/rx200_meshes/rx200_7_gripper_prop.stl" scale="0.001 0.001 0.001"/>
+        <mesh filename="package://robot_description/meshes/arm/arm/rx200_meshes/rx200_7_gripper_prop.stl" scale="0.001 0.001 0.001"/>
       </geometry>
       <material name="interbotix_black"/>
@@ -269,5 +269,5 @@
       <origin rpy="0 0 ${pi/2}" xyz="-0.0685 0 0"/>
       <geometry>
-        <mesh filename="package://interbotix_xsarm_descriptions/meshes/rx200_meshes/rx200_7_gripper_prop.stl" scale="0.001 0.001 0.001"/>
+        <mesh filename="package://robot_description/meshes/arm/arm/rx200_meshes/rx200_7_gripper_prop.stl" scale="0.001 0.001 0.001"/>
       </geometry>
     </collision>
@@ -290,5 +290,5 @@
         <origin rpy="0 0 0" xyz="0 0 0"/>
         <geometry>
-          <mesh filename="package://interbotix_xsarm_descriptions/meshes/rx200_meshes/rx200_10_ar_tag.stl" scale="0.001 0.001 0.001"/>
+          <mesh filename="package://robot_description/meshes/arm/arm/rx200_meshes/rx200_10_ar_tag.stl" scale="0.001 0.001 0.001"/>
         </geometry>
         <material name="interbotix_black"/>
@@ -297,5 +297,5 @@
         <origin rpy="0 0 0" xyz="0 0 0"/>
         <geometry>
-          <mesh filename="package://interbotix_xsarm_descriptions/meshes/rx200_meshes/rx200_10_ar_tag.stl" scale="0.001 0.001 0.001"/>
+          <mesh filename="package://robot_description/meshes/arm/arm/rx200_meshes/rx200_10_ar_tag.stl" scale="0.001 0.001 0.001"/>
         </geometry>
       </collision>
@@ -319,5 +319,5 @@
         <origin rpy="0 0 ${pi/2}" xyz="-0.063 0 0"/>
         <geometry>
-          <mesh filename="package://interbotix_xsarm_descriptions/meshes/rx200_meshes/rx200_8_gripper_bar.stl" scale="0.001 0.001 0.001"/>
+          <mesh filename="package://robot_description/meshes/arm/arm/rx200_meshes/rx200_8_gripper_bar.stl" scale="0.001 0.001 0.001"/>
         </geometry>
         <material name="interbotix_black"/>
@@ -326,5 +326,5 @@
         <origin rpy="0 0 ${pi/2}" xyz="-0.063 0 0"/>
         <geometry>
-          <mesh filename="package://interbotix_xsarm_descriptions/meshes/rx200_meshes/rx200_8_gripper_bar.stl" scale="0.001 0.001 0.001"/>
+          <mesh filename="package://robot_description/meshes/arm/arm/rx200_meshes/rx200_8_gripper_bar.stl" scale="0.001 0.001 0.001"/>
         </geometry>
       </collision>
@@ -370,5 +370,5 @@
           <origin rpy="${pi} ${pi} 0" xyz="0 0.005 0"/>
           <geometry>
-            <mesh filename="package://interbotix_xsarm_descriptions/meshes/rx200_meshes/rx200_9_gripper_finger.stl" scale="0.001 0.001 0.001"/>
+            <mesh filename="package://robot_description/meshes/arm/arm/rx200_meshes/rx200_9_gripper_finger.stl" scale="0.001 0.001 0.001"/>
           </geometry>
           <material name="interbotix_black"/>
@@ -377,5 +377,5 @@
           <origin rpy="${pi} ${pi} 0" xyz="0 0.005 0"/>
           <geometry>
-            <mesh filename="package://interbotix_xsarm_descriptions/meshes/rx200_meshes/rx200_9_gripper_finger.stl" scale="0.001 0.001 0.001"/>
+            <mesh filename="package://robot_description/meshes/arm/arm/rx200_meshes/rx200_9_gripper_finger.stl" scale="0.001 0.001 0.001"/>
           </geometry>
         </collision>
@@ -410,5 +410,5 @@
           <origin rpy="0 ${pi} 0" xyz="0 -0.005 0"/>
           <geometry>
-            <mesh filename="package://interbotix_xsarm_descriptions/meshes/rx200_meshes/rx200_9_gripper_finger.stl" scale="0.001 0.001 0.001"/>
+            <mesh filename="package://robot_description/meshes/arm/arm/rx200_meshes/rx200_9_gripper_finger.stl" scale="0.001 0.001 0.001"/>
           </geometry>
           <material name="interbotix_black"/>
@@ -417,5 +417,5 @@
           <origin rpy="0 ${pi} 0" xyz="0 -0.005 0"/>
           <geometry>
-            <mesh filename="package://interbotix_xsarm_descriptions/meshes/rx200_meshes/rx200_9_gripper_finger.stl" scale="0.001 0.001 0.001"/>
+            <mesh filename="package://robot_description/meshes/arm/arm/rx200_meshes/rx200_9_gripper_finger.stl" scale="0.001 0.001 0.001"/>
           </geometry>
         </collision>

File: src/robot_description/urdf/main/base.urdf.xacro (robot description, xacro)
@@ -114,5 +114,5 @@
          base_footprint + base_link + baseup_link stacks up), mounted
          HORIZONTAL (pitch = 0). Matches the sim URDF
-         (my_robot_nav/urdf/my_car.urdf.xacro) exactly so TF →
+         (robot_description/urdf/sim/my_car.urdf.xacro) exactly so TF →
          world-projection of YOLO detections is identical between sim
          and real. Previously the URDF had pitch = 0.562 rad (32°
@@ -123,5 +123,4 @@
       <origin xyz="0.149 0 1.272" rpy="0 0 0"/>
     </xacro:sensor_d435i>
-</robot>
   <!-- <joint name="camera_joint" type="fixed">
     <parent link="baseup_link"/>  <child link="camera_link"/>
@@ -134,2 +133,3 @@
   </visual>
 </link> -->
+</robot>
