Commit message: updated error handling ; reorganized robot urdf with arm

File: src/robot_description/urdf/sim/my_car_rx200.urdf.xacro (robot description, xacro)
@@ -1,7 +1,440 @@
 <?xml version="1.0"?>
-<robot name="omni_robot_rx200" xmlns:xacro="http://ros.org/wiki/xacro">
-  <!-- RX200 variant of the shared simulation robot. All chassis, sensor,
-       wheel, and Gazebo definitions come from my_car.urdf.xacro. -->
+<robot name="omni_robot" xmlns:xacro="http://ros.org/wiki/xacro">
+  <!-- Select the manipulator while keeping one shared mobile-base model. -->
+  <!-- RX200 is the default arm; pass arm_model:=piper for the legacy Piper. -->
   <xacro:arg name="arm_model" default="rx200"/>
-  <xacro:include filename="$(find robot_description)/urdf/sim/my_car.urdf.xacro"/>
+  <!-- The RX200 mount is 75 mm farther along +X than the original Piper
+       mount (0.037 + 0.075 = 0.112 m). -->
+  <xacro:property name="arm_mount_x"
+                  value="${0.112 if '$(arg arm_model)' == 'rx200' else 0.037}"/>
+  <!-- Create the reusable xacro module for Agilex Piper X arm self-collision. -->
+  <xacro:arg name="enable_piper_self_collision" default="true"/>
+  <!-- Frame enabled by default; pass enable_aluminium_frame:=false to disable. -->
+  <xacro:arg name="enable_aluminium_frame" default="true"/>
+  <!-- Piper's standalone world joint is disabled because arm_base_link is
+       mounted to this mobile base. -->
+  <xacro:arg name="piper_standalone" default="false"/>
+  <!-- This model supplies its own rendered D435i and Gazebo sensor below. -->
+  <xacro:arg name="piper_include_arm_camera" default="false"/>
+  <xacro:if value="${'$(arg arm_model)' == 'piper'}">
+    <xacro:include filename="$(find agx_arm_description)/agx_arm_urdf/piper/urdf/piper_with_gripper_description.xacro"/>
+  </xacro:if>
+  <!-- RX200 uses namespaced links such as rx200/base_link. Its description
+       defaults to use_world_frame=false, allowing this model to mount it. -->
+  <xacro:if value="${'$(arg arm_model)' == 'rx200'}">
+    <xacro:include filename="$(find robot_description)/urdf/arm/rx200.urdf.xacro"/>
+  </xacro:if>
+  <!-- Register piper_gazebo_self_collision only when Piper is selected. -->
+  <xacro:if value="${'$(arg arm_model)' == 'piper'}">
+    <xacro:include filename="$(find agx_arm_description)/agx_arm_urdf/piper/urdf/piper_self_collision.gazebo.xacro"/>
+  </xacro:if>
+  <!-- Reuse the real D435i frame tree and the portable eye-in-hand wrapper so
+       simulation and hardware publish the same optical frame names. -->
+  <xacro:include filename="$(find robot_description)/urdf/vision_voice/realsense_camera/d435i_eye_in_hand.urdf.xacro"/>
+  <!-- Structural aluminium profile assembly (30 x 30 mm). -->
+  <xacro:include filename="$(find robot_description)/urdf/sim/aluminium_3030_frame.urdf.xacro"/>
+  <material name="gray">
+    <color rgba="0.5 0.5 0.5 1"/>
+  </material>
+  <material name="black">
+    <color rgba="0 0 0 1"/>
+  </material>
+  <material name="white">
+    <color rgba="1 1 1 1"/>
+  </material>
+  <material name="blue">
+    <color rgba="0 0 1 1"/>
+  </material>
+  <!-- Base Footprint (ROOT) -->
+  <link name="base_footprint">
+    <visual>
+      <geometry>
+        <box size="0.001 0.001 0.001"/>
+      </geometry>
+      <material name="black"/>
+    </visual>
+  </link>
+  <!-- Base Link — uses the octagonal chassis mesh (32 triangles =
+       octagonal prism) shared with the real robot at
+       robot_description/urdf/main/base.urdf.xacro, so the Gazebo
+       silhouette matches the physical platform. Collision is a
+       circumscribing cylinder (r=0.30) to avoid ragged mesh
+       collisions with the mecanum drive. -->
+  <link name="base_link">
+    <visual>
+      <geometry>
+        <mesh filename="package://robot_description/urdf/main/meshes/base_link.stl"/>
+      </geometry>
+      <material name="gray"/>
+    </visual>
+    <collision>
+      <geometry>
+        <cylinder radius="0.30" length="0.02441"/>
+      </geometry>
+    </collision>
+    <inertial>
+      <mass value="2.0"/>
+      <origin xyz="0 0 0"/>
+      <inertia ixx="0.035" ixy="0" ixz="0" iyy="0.035" iyz="0" izz="0.07"/>
+    </inertial>
+  </link>
+  <joint name="base_footprint_joint" type="fixed">
+    <parent link="base_footprint"/>
+    <child link="base_link"/>
+    <origin xyz="0 0 0.04667" rpy="0 0 0"/>
+  </joint>
+  <!-- Base Up Link — same shared octagonal-top mesh as the real robot. -->
+  <link name="baseup_link">
+    <visual>
+      <geometry>
+        <mesh filename="package://robot_description/urdf/main/meshes/baseup_link.stl"/>
+      </geometry>
+      <material name="white"/>
+    </visual>
+    <collision>
+      <geometry>
+        <cylinder radius="0.30" length="0.03136"/>
+      </geometry>
+    </collision>
+    <inertial>
+      <mass value="1.0"/>
+      <origin xyz="0 0 0"/>
+      <inertia ixx="0.014" ixy="0" ixz="0" iyy="0.014" iyz="0" izz="0.027"/>
+    </inertial>
+  </link>
+  <joint name="baseup_joint" type="fixed">
+    <parent link="base_link"/>
+    <child link="baseup_link"/>
+    <origin xyz="0 0 0.04068" rpy="0 0 0"/>
+  </joint>
+  <!-- Wheel Macro -->
+  <xacro:macro name="omni_wheel" params="wheel_name x y z roll pitch yaw">
+    <link name="${wheel_name}">
+      <visual>
+        <geometry>
+          <cylinder radius="0.05" length="0.03804"/>
+        </geometry>
+        <!-- Rotate cylinder so axis (Z) aligns with Y -->
+        <origin xyz="0 0 0" rpy="1.5708 0 0"/>
+        <material name="black"/>
+      </visual>
+      <collision>
+        <geometry>
+          <cylinder radius="0.05" length="0.03804"/>
+        </geometry>
+        <!-- Collision follows Physics (Parallel) for smooth rolling -->
+        <origin xyz="0 0 0" rpy="1.5708 0 0"/>
+      </collision>
+      <inertial>
+        <mass value="0.5"/>
+        <origin xyz="0 0 0"/>
+        <inertia ixx="0.0004" ixy="0" ixz="0" iyy="0.0004" iyz="0" izz="0.0006"/>
+      </inertial>
+    </link>
+    <!-- Omni-roller friction model: high grip in the wheel's rolling
+         direction (mu1) + zero lateral grip (mu2) lets the wheel
+         slide freely perpendicular to its rolling axis. Without this,
+         the 4 wheels at ±45° yaw would fight each other and the
+         chassis would skid / lock. `fdir1` picks the primary
+         friction direction in the link frame; for the cylinder
+         rotated by rpy=(π/2, 0, 0), the rolling direction is link-X.
+         Setting min_depth pads the contact so ODE doesn't chatter
+         with such a small wheel radius. -->
+    <gazebo reference="${wheel_name}">
+      <mu1>1.0</mu1>
+      <mu2>0.0</mu2>
+      <fdir1>1 0 0</fdir1>
+      <kp>1e7</kp>
+      <kd>1.0</kd>
+      <minDepth>0.001</minDepth>
+      <maxVel>1.0</maxVel>
+    </gazebo>
+    <joint name="joint_${wheel_name}" type="continuous">
+      <parent link="base_link"/>
+      <child link="${wheel_name}"/>
+      <origin xyz="${x} ${y} ${z}" rpy="${roll} ${pitch} ${yaw}"/>
+      <axis xyz="0 1 0"/>
+    </joint>
+  </xacro:macro>
+  <!-- Wheels physically yawed ±45° — matches the real robot's 4-wheel
+       X-drive omni layout exactly (see base.urdf.xacro). The
+       `MecanumDrive` plugin's internal IK happens to be identical to the
+       X-drive analytical IK used by the navigation base controller
+       (both:  w = (vx ± vy ± (lx+ly)·ω)/R), so the plugin's
+       wheel-velocity commands are equivalent to real firmware commands.
+       What makes the 45° layout *physically correct* in Gazebo is the
+       per-wheel friction model (<gazebo reference="…"> blocks below):
+       mu2=0 permits the lateral slip that a real omni roller provides,
+       without which the four wheels would fight each other and the
+       chassis would skid / lock up. -->
+  <xacro:omni_wheel wheel_name="Rear_Left"   x="-0.1842" y=" 0.1842" z="0" roll="0" pitch="0" yaw="+0.785398"/>
+  <xacro:omni_wheel wheel_name="Front_Right" x=" 0.1842" y="-0.1842" z="0" roll="0" pitch="0" yaw="+0.785398"/>
+  <xacro:omni_wheel wheel_name="Front_Left"  x=" 0.1842" y=" 0.1842" z="0" roll="0" pitch="0" yaw="-0.785398"/>
+  <xacro:omni_wheel wheel_name="Rear_Right"  x="-0.1842" y="-0.1842" z="0" roll="0" pitch="0" yaw="-0.785398"/>
+  <!-- Lidar Link -->
+  <link name="lidar_link">
+    <visual>
+      <geometry>
+        <cylinder radius="0.03785" length="0.0413"/>
+      </geometry>
+      <material name="blue"/>
+    </visual>
+    <collision>
+      <geometry>
+        <cylinder radius="0.03785" length="0.0413"/>
+      </geometry>
+    </collision>
+    <inertial>
+      <mass value="0.2"/>
+      <origin xyz="0 0 0"/>
+      <inertia ixx="0.0001" ixy="0" ixz="0" iyy="0.0001" iyz="0" izz="0.0001"/>
+    </inertial>
+  </link>
+  <joint name="lidar_joint" type="fixed">
+    <parent link="baseup_link"/>
+    <child link="lidar_link"/>
+    <origin xyz="0.137 0 0.0335" rpy="0 0 0"/>
+  </joint>
+  <!-- Arm mount: the RX200 is at x=0.112 m; the legacy Piper remains at
+       x=0.037 m. Both arm bases are 0.445 m above baseup_link. -->
+  <xacro:if value="${'$(arg arm_model)' == 'piper'}">
+    <joint name="arm_base_joint" type="fixed">
+      <parent link="baseup_link"/>
+      <child link="arm_base_link"/>
+      <origin xyz="${arm_mount_x} 0 0.445" rpy="0 0 0"/>
+    </joint>
+  </xacro:if>
+  <xacro:if value="${'$(arg arm_model)' == 'rx200'}">
+    <joint name="arm_base_joint" type="fixed">
+      <parent link="baseup_link"/>
+      <child link="rx200/base_link"/>
+      <origin xyz="${arm_mount_x} 0 0.445" rpy="0 0 0"/>
+    </joint>
+  </xacro:if>
+  <!--
+    30 x 30 mm aluminium chassis (dimensions are in metres).
+    red:  two 1.33 m bars at y=+/-0.125, behind the arm at camera x=-0.121.
+          The bars start at the lidar_link origin height, z=0.0335.
+    blue: one 0.25 m crossbar between the two red posts at the top.
+    green: a 0.30 m rectangle extending forward (+X), with front legs
+           stopping 15 mm below the arm-base-link origin (z=0.445).
+    yellow: centre post directly beneath the selected arm base.
+    All x, y, z values are in the baseup_link coordinate frame.
+    The red/camera x parameter and the lidar frame height below match
+    THIS simulation file, not necessarily hardware mounting coordinates.
+  -->
+  <xacro:if value="$(arg enable_aluminium_frame)">
+    <xacro:aluminium_3030_frame
+        parent="baseup_link"
+        prefix="alu3030"
+        rear_x="-0.121"
+        half_width="0.125"
+        forward_length="0.30"
+        red_height="1.113"
+        bottom_z="0.0335"
+        arm_x="${arm_mount_x}"
+        arm_base_z="0.445"
+        arm_clearance="0.015"
+        profile_size="0.030"
+        wall_thickness="0.002"
+        aluminium_density="2700.0"/>
+  </xacro:if>
+  <!-- Description for self_collision of agx_piper -->
+  <xacro:if value="${'$(arg arm_model)' == 'piper'}">
+    <xacro:piper_gazebo_self_collision
+      enabled="$(arg enable_piper_self_collision)"/>
+  </xacro:if>
+  <!-- Real-robot D435i mount. The macro supplies camera_link plus nominal
+       color/depth/infrared optical frames for simulation. -->
+  <xacro:sensor_d435i parent="baseup_link" name="camera"
+                       use_nominal_extrinsics="true">
+    <origin xyz="-0.121 0 1.272" rpy="0 0 0"/>
+  </xacro:sensor_d435i>
+  <!-- Piper eye-in-hand D435i. For another arm, reuse this macro with its
+       tool/flange link as `parent` and replace only this calibrated origin.
+       The sensor macro defines arm_camera_link at the physical camera centre,
+       so this bottom-screw origin places that centre 0.05 m along -X, 0.025 m
+       along +Y, and 0.05 m along +Z from the joint6/link6 TF. -->
+  <xacro:if value="${'$(arg arm_model)' == 'piper'}">
+    <xacro:d435i_eye_in_hand parent="link6" name="arm_camera"
+                             use_nominal_extrinsics="true"
+                             gazebo_sensor_name="arm_rgbd_camera"
+                             topic="/arm_camera/arm_camera">
+      <origin xyz="-0.0375 0.0075 0.0394" rpy="0 ${3 * pi / 2} 0"/>
+    </xacro:d435i_eye_in_hand>
+  </xacro:if>
+  <!-- Gazebo Plugins and Sensors.
+       This machine runs ign-gazebo 6, whose system plugins still use
+       the ignition::gazebo::systems::* class names even when the
+       filename aliases are gz-sim-*. -->
+  <gazebo>
+    <!-- Drive Control Only (Odom is inaccurate for X-Drive) -->
+    <plugin
+      filename="gz-sim-mecanum-drive-system"
+      name="ignition::gazebo::systems::MecanumDrive">
+      <front_left_joint>joint_Front_Left</front_left_joint>
+      <front_right_joint>joint_Front_Right</front_right_joint>
+      <back_left_joint>joint_Rear_Left</back_left_joint>
+      <back_right_joint>joint_Rear_Right</back_right_joint>
+      <wheel_separation>0.3684</wheel_separation>
+      <wheelbase>0.3684</wheelbase>
+      <wheel_radius>0.05</wheel_radius>
+      <min_acceleration>-10</min_acceleration>
+      <max_acceleration>10</max_acceleration>
+      <topic>cmd_vel</topic>
+      <!-- Disable Plugin Odom by diverting to trash topics -->
+      <odom_topic>odom_trash</odom_topic>
+      <tf_topic>tf_trash</tf_topic>
+      <frame_id>odom</frame_id>
+      <child_frame_id>base_footprint</child_frame_id>
+    </plugin>
+    <!-- Ground Truth Odometry (Perfect Localization) -->
+    <plugin
+      filename="gz-sim-odometry-publisher-system"
+      name="ignition::gazebo::systems::OdometryPublisher">
+      <odom_frame>odom</odom_frame>
+      <robot_base_frame>base_footprint</robot_base_frame>
+      <odom_topic>odometry</odom_topic>
+      <tf_topic>tf</tf_topic>
+      <dimensions>2</dimensions> <!-- 2D Odom -->
+      <odom_publish_frequency>50</odom_publish_frequency>
+    </plugin>
+    <plugin
+      filename="gz-sim-joint-state-publisher-system"
+      name="ignition::gazebo::systems::JointStatePublisher">
+      <topic>/joint_states</topic>
+    </plugin>
+    <xacro:if value="${'$(arg arm_model)' == 'piper'}">
+      <plugin
+        filename="libignition-gazebo-joint-trajectory-controller-system.so"
+        name="ignition::gazebo::systems::JointTrajectoryController">
+        <topic>/piper/arm_joint_trajectory</topic>
+        <joint_name>joint1</joint_name>
+        <initial_position>0.0</initial_position>
+        <position_p_gain>80</position_p_gain>
+        <position_i_gain>0.1</position_i_gain>
+        <position_d_gain>8</position_d_gain>
+        <position_i_min>-2</position_i_min>
+        <position_i_max>2</position_i_max>
+        <position_cmd_min>-100</position_cmd_min>
+        <position_cmd_max>100</position_cmd_max>
+        <joint_name>joint2</joint_name>
+        <initial_position>0.0</initial_position>
+        <position_p_gain>80</position_p_gain>
+        <position_i_gain>0.1</position_i_gain>
+        <position_d_gain>8</position_d_gain>
+        <position_i_min>-2</position_i_min>
+        <position_i_max>2</position_i_max>
+        <position_cmd_min>-100</position_cmd_min>
+        <position_cmd_max>100</position_cmd_max>
+        <joint_name>joint3</joint_name>
+        <initial_position>0.0</initial_position>
+        <position_p_gain>70</position_p_gain>
+        <position_i_gain>0.1</position_i_gain>
+        <position_d_gain>7</position_d_gain>
+        <position_i_min>-2</position_i_min>
+        <position_i_max>2</position_i_max>
+        <position_cmd_min>-100</position_cmd_min>
+        <position_cmd_max>100</position_cmd_max>
+        <joint_name>joint4</joint_name>
+        <initial_position>0.0</initial_position>
+        <position_p_gain>50</position_p_gain>
+        <position_i_gain>0.05</position_i_gain>
+        <position_d_gain>5</position_d_gain>
+        <position_i_min>-1</position_i_min>
+        <position_i_max>1</position_i_max>
+        <position_cmd_min>-50</position_cmd_min>
+        <position_cmd_max>50</position_cmd_max>
+        <joint_name>joint5</joint_name>
+        <initial_position>0.0</initial_position>
+        <position_p_gain>40</position_p_gain>
+        <position_i_gain>0.05</position_i_gain>
+        <position_d_gain>4</position_d_gain>
+        <position_i_min>-1</position_i_min>
+        <position_i_max>1</position_i_max>
+        <position_cmd_min>-40</position_cmd_min>
+        <position_cmd_max>40</position_cmd_max>
+        <joint_name>joint6</joint_name>
+        <initial_position>0.0</initial_position>
+        <position_p_gain>30</position_p_gain>
+        <position_i_gain>0.02</position_i_gain>
+        <position_d_gain>3</position_d_gain>
+        <position_i_min>-1</position_i_min>
+        <position_i_max>1</position_i_max>
+        <position_cmd_min>-30</position_cmd_min>
+        <position_cmd_max>30</position_cmd_max>
+      </plugin>
+      <plugin
+        filename="libignition-gazebo-joint-trajectory-controller-system.so"
+        name="ignition::gazebo::systems::JointTrajectoryController">
+        <topic>/piper/gripper_joint_trajectory</topic>
+        <joint_name>gripper</joint_name>
+        <initial_position>0.0</initial_position>
+        <position_p_gain>25</position_p_gain>
+        <position_i_gain>0.02</position_i_gain>
+        <position_d_gain>2</position_d_gain>
+        <position_i_min>-0.5</position_i_min>
+        <position_i_max>0.5</position_i_max>
+        <position_cmd_min>-10</position_cmd_min>
+        <position_cmd_max>10</position_cmd_max>
+      </plugin>
+    </xacro:if>
+  </gazebo>
+  <gazebo reference="lidar_link">
+    <sensor name="lidar" type="gpu_lidar">
+      <pose>0 0 0 0 0 0</pose>
+      <always_on>true</always_on>
+      <visualize>true</visualize>
+      <topic>/scan</topic>
+      <update_rate>10</update_rate>
+      <gz_frame_id>lidar_link</gz_frame_id>
+      <ray>
+        <scan>
+          <horizontal>
+            <samples>360</samples>
+            <resolution>1</resolution>
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