Commit message: updated object placement in gazebo world ; included sts hardware interface from intergration team ; added d435 on arm joint 6 ; gpsr sequence modifications

File: src/robot_description/urdf/sim/my_car.urdf.xacro (robot description, xacro)
@@ -10,4 +10,6 @@
        because arm_base_link is mounted to this mobile base. -->
   <xacro:arg name="piper_standalone" default="false"/>
+  <!-- This model supplies its own rendered D435i and Gazebo sensor below. -->
+  <xacro:arg name="piper_include_arm_camera" default="false"/>
   <xacro:if value="${'$(arg arm_model)' == 'piper'}">
     <xacro:include filename="$(find agx_arm_description)/agx_arm_urdf/piper/urdf/piper_with_gripper_description.xacro"/>
@@ -242,4 +244,14 @@
     <origin xyz="-0.121 0 1.272" rpy="0 0 0"/>
   </xacro:sensor_d435i>
+  <!-- Piper eye-in-hand D435i. The sensor macro defines arm_camera_link at
+       the physical camera centre, so compensate for its bottom-screw origin
+       to place that centre 0.05 m along -X, 0.025 m along +Y, and 0.05 m
+       along +Z from the joint6/link6 TF. -->
+  <xacro:if value="${'$(arg arm_model)' == 'piper'}">
+    <xacro:sensor_d435i parent="link6" name="arm_camera"
+                         use_nominal_extrinsics="true">
+      <origin xyz="-0.0375 0.0075 0.0394" rpy="0 ${3 * pi / 2} 0"/>
+    </xacro:sensor_d435i>
+  </xacro:if>
   <!-- Gazebo Plugins and Sensors.
        This machine runs ign-gazebo 6, whose system plugins still use
@@ -283,4 +295,79 @@
       <topic>/joint_states</topic>
     </plugin>
+    <xacro:if value="${'$(arg arm_model)' == 'piper'}">
+      <plugin
+        filename="libignition-gazebo-joint-trajectory-controller-system.so"
+        name="ignition::gazebo::systems::JointTrajectoryController">
+        <topic>/piper/arm_joint_trajectory</topic>
+        <joint_name>joint1</joint_name>
+        <initial_position>0.0</initial_position>
+        <position_p_gain>80</position_p_gain>
+        <position_i_gain>0.1</position_i_gain>
+        <position_d_gain>8</position_d_gain>
+        <position_i_min>-2</position_i_min>
+        <position_i_max>2</position_i_max>
+        <position_cmd_min>-100</position_cmd_min>
+        <position_cmd_max>100</position_cmd_max>
+        <joint_name>joint2</joint_name>
+        <initial_position>0.0</initial_position>
+        <position_p_gain>80</position_p_gain>
+        <position_i_gain>0.1</position_i_gain>
+        <position_d_gain>8</position_d_gain>
+        <position_i_min>-2</position_i_min>
+        <position_i_max>2</position_i_max>
+        <position_cmd_min>-100</position_cmd_min>
+        <position_cmd_max>100</position_cmd_max>
+        <joint_name>joint3</joint_name>
+        <initial_position>0.0</initial_position>
+        <position_p_gain>70</position_p_gain>
+        <position_i_gain>0.1</position_i_gain>
+        <position_d_gain>7</position_d_gain>
+        <position_i_min>-2</position_i_min>
+        <position_i_max>2</position_i_max>
+        <position_cmd_min>-100</position_cmd_min>
+        <position_cmd_max>100</position_cmd_max>
+        <joint_name>joint4</joint_name>
+        <initial_position>0.0</initial_position>
+        <position_p_gain>50</position_p_gain>
+        <position_i_gain>0.05</position_i_gain>
+        <position_d_gain>5</position_d_gain>
+        <position_i_min>-1</position_i_min>
+        <position_i_max>1</position_i_max>
+        <position_cmd_min>-50</position_cmd_min>
+        <position_cmd_max>50</position_cmd_max>
+        <joint_name>joint5</joint_name>
+        <initial_position>0.0</initial_position>
+        <position_p_gain>40</position_p_gain>
+        <position_i_gain>0.05</position_i_gain>
+        <position_d_gain>4</position_d_gain>
+        <position_i_min>-1</position_i_min>
+        <position_i_max>1</position_i_max>
+        <position_cmd_min>-40</position_cmd_min>
+        <position_cmd_max>40</position_cmd_max>
+        <joint_name>joint6</joint_name>
+        <initial_position>0.0</initial_position>
+        <position_p_gain>30</position_p_gain>
+        <position_i_gain>0.02</position_i_gain>
+        <position_d_gain>3</position_d_gain>
+        <position_i_min>-1</position_i_min>
+        <position_i_max>1</position_i_max>
+        <position_cmd_min>-30</position_cmd_min>
+        <position_cmd_max>30</position_cmd_max>
+      </plugin>
+      <plugin
+        filename="libignition-gazebo-joint-trajectory-controller-system.so"
+        name="ignition::gazebo::systems::JointTrajectoryController">
+        <topic>/piper/gripper_joint_trajectory</topic>
+        <joint_name>gripper</joint_name>
+        <initial_position>0.0</initial_position>
+        <position_p_gain>25</position_p_gain>
+        <position_i_gain>0.02</position_i_gain>
+        <position_d_gain>2</position_d_gain>
+        <position_i_min>-0.5</position_i_min>
+        <position_i_max>0.5</position_i_max>
+        <position_cmd_min>-10</position_cmd_min>
+        <position_cmd_max>10</position_cmd_max>
+      </plugin>
+    </xacro:if>
   </gazebo>
   <gazebo reference="lidar_link">
@@ -341,3 +428,29 @@
     </sensor>
   </gazebo>
+  <gazebo reference="arm_camera_link">
+    <sensor name="arm_rgbd_camera" type="rgbd_camera">
+      <always_on>true</always_on>
+      <update_rate>30</update_rate>
+      <topic>/arm_camera/arm_camera</topic>
+      <gz_frame_id>arm_camera_color_optical_frame</gz_frame_id>
+      <camera>
+        <horizontal_fov>1.2112</horizontal_fov>
+        <image>
+          <width>640</width>
+          <height>480</height>
+          <format>R8G8B8</format>
+        </image>
+        <clip>
+          <near>0.10</near>
+          <far>5.0</far>
+        </clip>
+        <depth_camera>
+          <clip>
+            <near>0.10</near>
+            <far>5.0</far>
+          </clip>
+        </depth_camera>
+      </camera>
+    </sensor>
+  </gazebo>
 </robot>

Commit message: unfinished fix on qwen based target selector + depth resolver on target ; configuration of simulation for dual axis head

File: src/robot_description/urdf/sim/my_car.urdf.xacro (robot description, xacro)
@@ -2,11 +2,27 @@
 <robot name="omni_robot" xmlns:xacro="http://ros.org/wiki/xacro">
   <!-- Select the manipulator while keeping one shared mobile-base model. -->
+  <!-- RX200 is the default arm; pass arm_model:=piper for the legacy Piper. -->
   <xacro:arg name="arm_model" default="piper"/>
+  <!-- The RX200 mount is 75 mm farther along +X than the original Piper
+       mount (0.037 + 0.075 = 0.112 m). -->
+  <xacro:property name="arm_mount_x"
+                  value="${0.112 if '$(arg arm_model)' == 'rx200' else 0.037}"/>
   <!-- Create the reusable xacro module for Agilex Piper X arm self-collision. -->
   <xacro:arg name="enable_piper_self_collision" default="true"/>
   <!-- Frame enabled by default; pass enable_aluminium_frame:=false to disable. -->
   <xacro:arg name="enable_aluminium_frame" default="true"/>
-  <!-- Piper is the default arm. Its standalone world joint is disabled
-       because arm_base_link is mounted to this mobile base. -->
+  <xacro:arg name="enable_head_gimbal" default="true"/>
+  <!-- Exactly one head controller backend may own the joints: gazebo, sts, none. -->
+  <xacro:arg name="head_control_backend" default="gazebo"/>
+  <xacro:arg name="head_serial_port" default="/dev/ttyACM0"/>
+  <xacro:arg name="head_use_mock" default="false"/>
+  <xacro:arg name="head_yaw_motor_id" default="1"/>
+  <xacro:arg name="head_pitch_motor_id" default="2"/>
+  <xacro:arg name="head_yaw_center_steps" default="2048"/>
+  <xacro:arg name="head_pitch_center_steps" default="2048"/>
+  <xacro:arg name="head_yaw_direction" default="1"/>
+  <xacro:arg name="head_pitch_direction" default="-1"/>
+  <!-- Piper's standalone world joint is disabled because arm_base_link is
+       mounted to this mobile base. -->
   <xacro:arg name="piper_standalone" default="false"/>
   <!-- This model supplies its own rendered D435i and Gazebo sensor below. -->
@@ -20,9 +36,13 @@
     <xacro:include filename="$(find robot_description)/urdf/arm/rx200.urdf.xacro"/>
   </xacro:if>
-  <!-- Register piper_gazebo_self_collision -->
-  <xacro:include filename="$(find agx_arm_description)/agx_arm_urdf/piper/urdf/piper_self_collision.gazebo.xacro"/>
-  <!-- Reuse the real D435i frame tree so simulation and hardware publish the
-       same camera_link/color/depth/infra optical frame names. -->
-  <xacro:include filename="$(find robot_description)/urdf/vision_voice/realsense_camera/_d435i.urdf.xacro"/>
+  <!-- Register piper_gazebo_self_collision only when Piper is selected. -->
+  <xacro:if value="${'$(arg arm_model)' == 'piper'}">
+    <xacro:include filename="$(find agx_arm_description)/agx_arm_urdf/piper/urdf/piper_self_collision.gazebo.xacro"/>
+  </xacro:if>
+  <!-- Reuse the real D435i frame tree and the portable eye-in-hand wrapper so
+       simulation and hardware publish the same optical frame names. -->
+  <xacro:include filename="$(find robot_description)/urdf/vision_voice/realsense_camera/d435i_eye_in_hand.urdf.xacro"/>
+  <xacro:include filename="$(find robot_description)/urdf/sim/head_assembly.urdf.xacro"/>
+  <xacro:include filename="$(find robot_description)/urdf/sim/head_sts_control.urdf.xacro"/>
   <!-- Structural aluminium profile assembly (30 x 30 mm). -->
   <xacro:include filename="$(find robot_description)/urdf/sim/aluminium_3030_frame.urdf.xacro"/>
@@ -189,11 +209,11 @@
     <origin xyz="0.137 0 0.0335" rpy="0 0 0"/>
   </joint>
-  <!-- Arm mount: 0.10 m behind the lidar along robot X, with the arm base
-       0.445 m above baseup_link. -->
+  <!-- Arm mount: the RX200 is at x=0.112 m; the legacy Piper remains at
+       x=0.037 m. Both arm bases are 0.445 m above baseup_link. -->
   <xacro:if value="${'$(arg arm_model)' == 'piper'}">
     <joint name="arm_base_joint" type="fixed">
       <parent link="baseup_link"/>
       <child link="arm_base_link"/>
-      <origin xyz="0.037 0 0.445" rpy="0 0 0"/>
+      <origin xyz="${arm_mount_x} 0 0.445" rpy="0 0 0"/>
     </joint>
   </xacro:if>
@@ -202,5 +222,5 @@
       <parent link="baseup_link"/>
       <child link="rx200/base_link"/>
-      <origin xyz="0.037 0 0.445" rpy="0 0 0"/>
+      <origin xyz="${arm_mount_x} 0 0.445" rpy="0 0 0"/>
     </joint>
   </xacro:if>
@@ -212,5 +232,5 @@
     green: a 0.30 m rectangle extending forward (+X), with front legs
            stopping 15 mm below the arm-base-link origin (z=0.445).
-    yellow: centre post directly beneath the arm base at x=0.037.
+    yellow: centre post directly beneath the selected arm base.
     All x, y, z values are in the baseup_link coordinate frame.
     The red/camera x parameter and the lidar frame height below match
@@ -226,5 +246,5 @@
         red_height="1.113"
         bottom_z="0.0335"
-        arm_x="0.037"
+        arm_x="${arm_mount_x}"
         arm_base_z="0.445"
         arm_clearance="0.015"
@@ -238,19 +258,39 @@
       enabled="$(arg enable_piper_self_collision)"/>
   </xacro:if>
-  <!-- Real-robot D435i mount. The macro supplies camera_link plus nominal
-       color/depth/infrared optical frames for simulation. -->
-  <xacro:sensor_d435i parent="baseup_link" name="camera"
-                       use_nominal_extrinsics="true">
-    <origin xyz="-0.121 0 1.272" rpy="0 0 0"/>
-  </xacro:sensor_d435i>
-  <!-- Piper eye-in-hand D435i. The sensor macro defines arm_camera_link at
-       the physical camera centre, so compensate for its bottom-screw origin
-       to place that centre 0.05 m along -X, 0.025 m along +Y, and 0.05 m
-       along +Z from the joint6/link6 TF. -->
+  <!-- The gimbal replaces the original fixed mast camera. The fallback keeps
+       exactly one camera tree when either the frame or gimbal is disabled. -->
+  <xacro:if value="${'$(arg enable_aluminium_frame)' == 'true' and '$(arg enable_head_gimbal)' == 'true'}">
+    <xacro:head_camera_assembly parent="alu3030_blue_camera_top"
+                                enable_gazebo="${'$(arg head_control_backend)' == 'gazebo'}"/>
+    <xacro:if value="${'$(arg head_control_backend)' == 'sts'}">
+      <xacro:head_sts_control
+          serial_port="$(arg head_serial_port)"
+          use_mock="$(arg head_use_mock)"
+          yaw_motor_id="$(arg head_yaw_motor_id)"
+          pitch_motor_id="$(arg head_pitch_motor_id)"
+          yaw_center_steps="$(arg head_yaw_center_steps)"
+          pitch_center_steps="$(arg head_pitch_center_steps)"
+          yaw_direction="$(arg head_yaw_direction)"
+          pitch_direction="$(arg head_pitch_direction)"/>
+    </xacro:if>
+  </xacro:if>
+  <xacro:unless value="${'$(arg enable_aluminium_frame)' == 'true' and '$(arg enable_head_gimbal)' == 'true'}">
+    <xacro:sensor_d435i parent="baseup_link" name
+                         use_nominal_extrinsics="true">
+      <origin xyz="-0.121 0 1.272" rpy="0 0 0"/>
+    </xacro:sensor_d435i>
+  </xacro:unless>
+  <!-- Piper eye-in-hand D435i. For another arm, reuse this macro with its
+       tool/flange link as `parent` and replace only this calibrated origin.
+       The sensor macro defines arm_camera_link at the physical camera centre,
+       so this bottom-screw origin places that centre 0.05 m along -X, 0.025 m
+       along +Y, and 0.05 m along +Z from the joint6/link6 TF. -->
   <xacro:if value="${'$(arg arm_model)' == 'piper'}">
-    <xacro:sensor_d435i parent="link6" name="arm_camera"
-                         use_nominal_extrinsics="true">
+    <xacro:d435i_eye_in_hand parent="link6" name="arm_camera"
+                             use_nominal_extrinsics="true"
+                             gazebo_sensor_name="arm_rgbd_camera"
+                             topic="/arm_camera/arm_camera">
       <origin xyz="-0.0375 0.0075 0.0394" rpy="0 ${3 * pi / 2} 0"/>
-    </xacro:sensor_d435i>
+    </xacro:d435i_eye_in_hand>
   </xacro:if>
   <!-- Gazebo Plugins and Sensors.
@@ -428,29 +468,3 @@
     </sensor>
   </gazebo>
-  <gazebo reference="arm_camera_link">
-    <sensor name="arm_rgbd_camera" type="rgbd_camera">
-      <always_on>true</always_on>
-      <update_rate>30</update_rate>
-      <topic>/arm_camera/arm_camera</topic>
-      <gz_frame_id>arm_camera_color_optical_frame</gz_frame_id>
-      <camera>
-        <horizontal_fov>1.2112</horizontal_fov>
-        <image>
-          <width>640</width>
-          <height>480</height>
-          <format>R8G8B8</format>
-        </image>
-        <clip>
-          <near>0.10</near>
-          <far>5.0</far>
-        </clip>
-        <depth_camera>
-          <clip>
-            <near>0.10</near>
-            <far>5.0</far>
-          </clip>
-        </depth_camera>
-      </camera>
-    </sensor>
-  </gazebo>
 </robot>

File: src/robot_description/urdf/sim/my_car_rx200.urdf.xacro (robot description, xacro)
@@ -12,4 +12,15 @@
   <!-- Frame enabled by default; pass enable_aluminium_frame:=false to disable. -->
   <xacro:arg name="enable_aluminium_frame" default="true"/>
+  <xacro:arg name="enable_head_gimbal" default="true"/>
+  <!-- Exactly one head controller backend may own the joints: gazebo, sts, none. -->
+  <xacro:arg name="head_control_backend" default="gazebo"/>
+  <xacro:arg name="head_serial_port" default="/dev/ttyACM0"/>
+  <xacro:arg name="head_use_mock" default="false"/>
+  <xacro:arg name="head_yaw_motor_id" default="1"/>
+  <xacro:arg name="head_pitch_motor_id" default="2"/>
+  <xacro:arg name="head_yaw_center_steps" default="2048"/>
+  <xacro:arg name="head_pitch_center_steps" default="2048"/>
+  <xacro:arg name="head_yaw_direction" default="1"/>
+  <xacro:arg name="head_pitch_direction" default="-1"/>
   <!-- Piper's standalone world joint is disabled because arm_base_link is
        mounted to this mobile base. -->
@@ -32,4 +43,6 @@
        simulation and hardware publish the same optical frame names. -->
   <xacro:include filename="$(find robot_description)/urdf/vision_voice/realsense_camera/d435i_eye_in_hand.urdf.xacro"/>
+  <xacro:include filename="$(find robot_description)/urdf/sim/head_assembly.urdf.xacro"/>
+  <xacro:include filename="$(find robot_description)/urdf/sim/head_sts_control.urdf.xacro"/>
   <!-- Structural aluminium profile assembly (30 x 30 mm). -->
   <xacro:include filename="$(find robot_description)/urdf/sim/aluminium_3030_frame.urdf.xacro"/>
@@ -245,10 +258,27 @@
       enabled="$(arg enable_piper_self_collision)"/>
   </xacro:if>
-  <!-- Real-robot D435i mount. The macro supplies camera_link plus nominal
-       color/depth/infrared optical frames for simulation. -->
-  <xacro:sensor_d435i parent="baseup_link" name="camera"
-                       use_nominal_extrinsics="true">
-    <origin xyz="-0.121 0 1.272" rpy="0 0 0"/>
-  </xacro:sensor_d435i>
+  <!-- The gimbal replaces the original fixed mast camera. The fallback keeps
+       exactly one camera tree when either the frame or gimbal is disabled. -->
+  <xacro:if value="${'$(arg enable_aluminium_frame)' == 'true' and '$(arg enable_head_gimbal)' == 'true'}">
+    <xacro:head_camera_assembly parent="alu3030_blue_camera_top"
+                                enable_gazebo="${'$(arg head_control_backend)' == 'gazebo'}"/>
+    <xacro:if value="${'$(arg head_control_backend)' == 'sts'}">
+      <xacro:head_sts_control
+          serial_port="$(arg head_serial_port)"
+          use_mock="$(arg head_use_mock)"
+          yaw_motor_id="$(arg head_yaw_motor_id)"
+          pitch_motor_id="$(arg head_pitch_motor_id)"
+          yaw_center_steps="$(arg head_yaw_center_steps)"
+          pitch_center_steps="$(arg head_pitch_center_steps)"
+          yaw_direction="$(arg head_yaw_direction)"
+          pitch_direction="$(arg head_pitch_direction)"/>
+    </xacro:if>
+  </xacro:if>
+  <xacro:unless value="${'$(arg enable_aluminium_frame)' == 'true' and '$(arg enable_head_gimbal)' == 'true'}">
+    <xacro:sensor_d435i parent="baseup_link" name="camera"
+                         use_nominal_extrinsics="true">
+      <origin xyz="-0.121 0 1.272" rpy="0 0 0"/>
+    </xacro:sensor_d435i>
+  </xacro:unless>
   <!-- Piper eye-in-hand D435i. For another arm, reuse this macro with its
        tool/flange link as `parent` and replace only this calibrated origin.
@@ -262,4 +292,16 @@
                              topic="/arm_camera/arm_camera">
       <origin xyz="-0.0375 0.0075 0.0394" rpy="0 ${3 * pi / 2} 0"/>
+    </xacro:d435i_eye_in_hand>
+  </xacro:if>
+  <!-- RX200 eye-in-hand D435i mounted at the wrist_rotate output. The
+       wrist_rotate joint's child is gripper_link; these coordinates are
+       relative to that link: +0.04 m in X and +0.05 m in Z. -->
+  <xacro:if value="${'$(arg arm_model)' == 'rx200'}">
+    <xacro:d435i_eye_in_hand parent="rx200/gripper_link"
+                             name="rx200_wrist_camera"
+                             use_nominal_extrinsics="true"
+                             gazebo_sensor_name="rx200_wrist_rgbd_camera"
+                             topic="/rx200_wrist_camera/rgbd">
+      <origin xyz="0.04 0 0.05" rpy="0 0 0"/>
     </xacro:d435i_eye_in_hand>
   </xacro:if>
@@ -371,4 +413,84 @@
         <joint_name>gripper</joint_name>
         <initial_position>0.0</initial_position>
+        <position_p_gain>25</position_p_gain>
+        <position_i_gain>0.02</position_i_gain>
+        <position_d_gain>2</position_d_gain>
+        <position_i_min>-0.5</position_i_min>
+        <position_i_max>0.5</position_i_max>
+        <position_cmd_min>-10</position_cmd_min>
+        <position_cmd_max>10</position_cmd_max>
+      </plugin>
+    </xacro:if>
+    <!-- RX200 trajectory controllers for Gazebo Sim. MoveIt sends
+         FollowJointTrajectory goals to a ROS action relay, which forwards
+         JointTrajectory messages to these native Gazebo controllers. -->
+    <xacro:if value="${'$(arg arm_model)' == 'rx200'}">
+      <plugin
+        filename="libignition-gazebo-joint-trajectory-controller-system.so"
+        name="ignition::gazebo::systems::JointTrajectoryController">
+        <topic>/rx200/arm_joint_trajectory</topic>
+        <joint_name>waist</joint_name>
+        <initial_position>0.0</initial_position>
+        <position_p_gain>80</position_p_gain>
+        <position_i_gain>0.1</position_i_gain>
+        <position_d_gain>8</position_d_gain>
+        <position_i_min>-2</position_i_min>
+        <position_i_max>2</position_i_max>
+        <position_cmd_min>-100</position_cmd_min>
+        <position_cmd_max>100</position_cmd_max>
+        <joint_name>shoulder</joint_name>
+        <initial_position>0.0</initial_position>
+        <position_p_gain>80</position_p_gain>
+        <position_i_gain>0.1</position_i_gain>
+        <position_d_gain>8</position_d_gain>
+        <position_i_min>-2</position_i_min>
+        <position_i_max>2</position_i_max>
+        <position_cmd_min>-100</position_cmd_min>
+        <position_cmd_max>100</position_cmd_max>
+        <joint_name>elbow</joint_name>
+        <initial_position>0.0</initial_position>
+        <position_p_gain>70</position_p_gain>
+        <position_i_gain>0.1</position_i_gain>
+        <position_d_gain>7</position_d_gain>
+        <position_i_min>-2</position_i_min>
+        <position_i_max>2</position_i_max>
+        <position_cmd_min>-100</position_cmd_min>
+        <position_cmd_max>100</position_cmd_max>
+        <joint_name>wrist_angle</joint_name>
+        <initial_position>0.0</initial_position>
+        <position_p_gain>50</position_p_gain>
+        <position_i_gain>0.05</position_i_gain>
+        <position_d_gain>5</position_d_gain>
+        <position_i_min>-1</position_i_min>
+        <position_i_max>1</position_i_max>
+        <position_cmd_min>-50</position_cmd_min>
+        <position_cmd_max>50</position_cmd_max>
+        <joint_name>wrist_rotate</joint_name>
+        <initial_position>0.0</initial_position>
+        <position_p_gain>40</position_p_gain>
+        <position_i_gain>0.05</position_i_gain>
+        <position_d_gain>4</position_d_gain>
+        <position_i_min>-1</position_i_min>
+        <position_i_max>1</position_i_max>
+        <position_cmd_min>-40</position_cmd_min>
+        <position_cmd_max>40</position_cmd_max>
+      </plugin>
+      <!-- Both finger joints are commanded explicitly because Gazebo Sim's
+           URDF-to-SDF mimic handling varies between Fortress releases. -->
+      <plugin
+        filename="libignition-gazebo-joint-trajectory-controller-system.so"
+        name="ignition::gazebo::systems::JointTrajectoryController">
+        <topic>/rx200/gripper_joint_trajectory</topic>
+        <joint_name>left_finger</joint_name>
+        <initial_position>0.037</initial_position>
+        <position_p_gain>25</position_p_gain>
+        <position_i_gain>0.02</position_i_gain>
+        <position_d_gain>2</position_d_gain>
+        <position_i_min>-0.5</position_i_min>
+        <position_i_max>0.5</position_i_max>
+        <position_cmd_min>-10</position_cmd_min>
+        <position_cmd_max>10</position_cmd_max>
+        <joint_name>right_finger</joint_name>
+        <initial_position>-0.037</initial_position>
         <position_p_gain>25</position_p_gain>
         <position_i_gain>0.02</position_i_gain>
